File: pcb/sonopi-dac.sch (EAGLE design)
At the start: 22 parts, among them J1 AV2-8.4-10GA, U1 PCM5122PW, U2 MCP1703AT-3302E/CB, X1 RASPI_BOARD_B+#_ZERO, X2 22.5792MHz, X3 24.576MHz

Commit message: fix a minor bug in schema
Connections:
- removed net EN44: X2.EN
- net EN41: now also X2.EN
Changed lines of the file:
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@@
 <label x="114.3" y="109.22" size="1.778" layer="95" rot="MR0"/>
+</segment>
+<segment>
+<pinref part="X2" gate="G$1" pin="EN"/>
+<wire x1="30.48" y1="60.96" x2="20.32" y2="60.96" width="0.1524" layer="91"/>
+<label x="20.32" y="60.96" size="1.778" layer="95"/>
 </segment>
 </net>
@@
 </segment>
 </net>
-<net name="EN44" class="0">
-<segment>
-<pinref part="X2" gate="G$1" pin="EN"/>
-<wire x1="30.48" y1="60.96" x2="20.32" y2="60.96" width="0.1524" layer="91"/>
-<label x="20.32" y="60.96" size="1.778" layer="95"/>
-</segment>
-</net>
 <net name="N$3" class="0">
 <segment>
@@
 </sheet>
 </sheets>
+<errors>
+</errors>
 </schematic>
 </drawing>

Commit message: fix a bug that a part of coupling capaciter does not be utilized
Parts:
- added C15, C16: 2.2nF/50V, rcl:C-EUC0603
- C11: value 0.1uF/100V -> 10uF/16V; device rcl:C-EUC0603 -> rcl:C-EUC3216
- C13, C14: value 2.2nF/50V -> 0.1uF/100V
Connections:
- net N$1 renamed VNEG
- net N$4 renamed CAPP
- net N$5 renamed CAPM
- removed net N$3: C13.2, J1.LEFT-CH, R1.2
- removed net N$6: C14.1, J1.RIGHT-CH, R2.2
- new net LCH: C15.2, J1.LEFT-CH, R1.2
- new net RCH: C16.1, J1.RIGHT-CH, R2.2
- net +3V3: now also C13.1, C14.1; no longer C11.1, C12.1
- net +3V3/A: now also C11.1, C12.1
- net GND: now also C13.2, C15.1, C16.2; no longer C13.1
Other:
- moved on the sheet: C10, C11, C12, C13, C14, C3, C4, C5, C6, C7, C8, C9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

Commit message: initial artwork done
Connections:
- net N$2 renamed LDOO
Changed lines of the file:
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@@
 </class>
 <class number="1" name="gnd" width="0.2" drill="0">
+<clearance class="1" value="0.1"/>
 </class>
 <class number="2" name="pwr" width="0.2" drill="0">
+<clearance class="2" value="0.1"/>
 </class>
 </classes>
@@
 </segment>
 </net>
-<net name="N$2" class="0">
+<net name="LDOO" class="0">
 <segment>
 <pinref part="U1" gate="G$1" pin="LDOO"/>

Commit message: add artwork design
Parts:
- removed X3: 24.576MHz, oscillator:OSC-3225
- added J2: RASPI_BOARD_B+#_ZERO, raspi-zero-i2s:RASPI_BOARD_B+#_ZERO
- X1: value RASPI_BOARD_B+#_ZERO -> 22.5792MHz; device raspi-zero-i2s:RASPI_BOARD_B+#_ZERO -> oscillator:OSC-3225
- X2: value 22.5792MHz -> 24.576MHz
Connections:
- net +3V3: now also J2.3V3_A, X1.VDD; no longer X1.3V3_A, X3.VDD
- net +5V: now also J2.5V0A, J2.5V0B; no longer X1.5V0A, X1.5V0B
- net BCLK: now also J2.GPIO18; no longer X1.GPIO18
- net DATA: now also J2.GPIO21; no longer X1.GPIO21
- net EN41: now also X1.EN; no longer X2.EN
- net EN48: now also X2.EN; no longer X3.EN
- net GND: now also J2.GND_A, J2.GND_B, J2.GND_H, X1.GND; no longer X1.GND_A, X1.GND_B, X1.GND_H, X3.GND
- net LRCLK: now also J2.GPIO19; no longer X1.GPIO19
- net SCL: now also J2.SCL; no longer X1.SCL
- net SCLK: now also X1.OUT; no longer X3.OUT
- net SDA: now also J2.SDA; no longer X1.SDA
Other:
- moved on the sheet: X2
Changed lines of the file:
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@@
 </classes>
 <parts>
-<part name="X1" library="raspi-zero-i2s" deviceset="RASPI_BOARD_B+#" device="_ZERO" package3d_urn="urn:adsk.eagle:package:7043377/3"/>
+<part name="J2" library="raspi-zero-i2s" library_urn="urn:adsk.eagle:library:15297902" deviceset="RASPI_BOARD_B+#" device="_ZERO" package3d_urn="urn:adsk.eagle:package:7043377/5"/>
 <part name="U2" library="SOT23_Module" deviceset="LDO-REGULATOR" device="" package3d_urn="urn:adsk.eagle:package:28534/2" value="MCP1703AT-3302E/CB"/>
 <part name="GND2" library="supply1" library_urn="urn:adsk.eagle:library:371" deviceset="GND" device=""/>
@@
 <part name="P+1" library="supply1" library_urn="urn:adsk.eagle:library:371" deviceset="+5V" device=""/>
 <part name="GND1" library="supply1" library_urn="urn:adsk.eagle:library:371" deviceset="GND" device=""/>
-<part name="U1" library="PCM5122" deviceset="PCM5122PW" device=""/>
+<part name="U1" library="PCM5122" library_urn="urn:adsk.eagle:library:15275669" deviceset="PCM5122PW" device="" package3d_urn="urn:adsk.eagle:package:15275672/2"/>
 <part name="+3V2" library="supply1" library_urn="urn:adsk.eagle:library:371" deviceset="+3V3" device=""/>
 <part name="C4" library="rcl" library_urn="urn:adsk.eagle:library:334" deviceset="C-EU" device="C0603" package3d_urn="urn:adsk.eagle:package:23616/2" value="0.1uF/100V"/>
@@
 <part name="C10" library="rcl" library_urn="urn:adsk.eagle:library:334" deviceset="C-EU" device="C0805" package3d_urn="urn:adsk.eagle:package:23617/2" value="2.2uF/25V"/>
 <part name="R1" library="rcl" library_urn="urn:adsk.eagle:library:334" deviceset="R-US_" device="R0603" package3d_urn="urn:adsk.eagle:package:23555/3" value="470Ω"/>
-<part name="X2" library="oscillator" deviceset="OSC" device="-3225" value="22.5792MHz"/>
-<part name="J1" library="RCA-jack" deviceset="2CH-RCA" device="AITENDO" value="AV2-8.4-10GA"/>
+<part name="X1" library="oscillator" library_urn="urn:adsk.eagle:library:15275959" deviceset="OSC" device="-3225" package3d_urn="urn:adsk.eagle:package:15275963/2" value="22.5792MHz"/>
+<part name="J1" library="RCA-jack" library_urn="urn:adsk.eagle:library:15327963" deviceset="2CH-RCA" device="AITENDO" package3d_urn="urn:adsk.eagle:package:15327967/3" value="AV2-8.4-10GA"/>
 <part name="+3V3" library="supply1" library_urn="urn:adsk.eagle:library:371" deviceset="+3V3" device=""/>
 <part name="C13" library="rcl" library_urn="urn:adsk.eagle:library:334" deviceset="C-EU" device="C0603" package3d_urn="urn:adsk.eagle:package:23616/2" value="0.1uF/100V"/>
 <part name="GND8" library="supply1" library_urn="urn:adsk.eagle:library:371" deviceset="GND" device=""/>
-<part name="X3" library="oscillator" deviceset="OSC" device="-3225" value="24.576MHz"/>
+<part name="X2" library="oscillator" library_urn="urn:adsk.eagle:library:15275959" deviceset="OSC" device="-3225" package3d_urn="urn:adsk.eagle:package:15275963/2" value="24.576MHz"/>
 <part name="+3V4" library="supply1" library_urn="urn:adsk.eagle:library:371" deviceset="+3V3" device=""/>
 <part name="C14" library="rcl" library_urn="urn:adsk.eagle:library:334" deviceset="C-EU" device="C0603" package3d_urn="urn:adsk.eagle:package:23616/2" value="0.1uF/100V"/>
@@
 </plain>
 <instances>
-<instance part="X1" gate="G$1" x="228.6" y="124.46" smashed="yes"/>
+<instance part="J2" gate="G$1" x="228.6" y="124.46" smashed="yes"/>
 <instance part="U2" gate="G$1" x="172.72" y="17.78" smashed="yes">
 <attribute name="NAME" x="147.32" y="45.72" size="1.778" layer="95" align="center"/>
@@
 <attribute name="VALUE" x="204.47" y="42.418" size="1.778" layer="96"/>
 </instance>
-<instance part="X2" gate="G$1" x="45.72" y="58.42" smashed="yes">
+<instance part="X1" gate="G$1" x="45.72" y="58.42" smashed="yes">
 <attribute name="NAME" x="45.72" y="66.04" size="1.778" layer="95" align="center"/>
 <attribute name="VALUE" x="45.72" y="53.34" size="1.778" layer="96" align="center"/>
@@
 <attribute name="VALUE" x="73.66" y="40.64" size="1.778" layer="96"/>
 </instance>
-<instance part="X3" gate="G$1" x="45.72" y="22.86" smashed="yes">
+<instance part="X2" gate="G$1" x="45.72" y="22.86" smashed="yes">
 <attribute name="NAME" x="45.72" y="30.48" size="1.778" layer="95" align="center"/>
 <attribute name="VALUE" x="45.72" y="17.78" size="1.778" layer="96" align="center"/>
@@
 <segment>
 <pinref part="P+1" gate="1" pin="+5V"/>
-<pinref part="X1" gate="G$1" pin="5V0A"/>
+<pinref part="J2" gate="G$1" pin="5V0A"/>
 <wire x1="220.98" y1="157.48" x2="220.98" y2="154.94" width="0.1524" layer="91"/>
-<pinref part="X1" gate="G$1" pin="5V0B"/>
+<pinref part="J2" gate="G$1" pin="5V0B"/>
 <wire x1="220.98" y1="154.94" x2="220.98" y2="152.4" width="0.1524" layer="91"/>
 <wire x1="220.98" y1="154.94" x2="223.52" y2="154.94" width="0.1524" layer="91"/>
@@
 </segment>
 <segment>
-<pinref part="X1" gate="G$1" pin="GND_A"/>
+<pinref part="J2" gate="G$1" pin="GND_A"/>
 <wire x1="243.84" y1="129.54" x2="251.46" y2="129.54" width="0.1524" layer="91"/>
 <wire x1="251.46" y1="129.54" x2="251.46" y2="127" width="0.1524" layer="91"/>
 <pinref part="GND1" gate="1" pin="GND"/>
-<pinref part="X1" gate="G$1" pin="GND_B"/>
+<pinref part="J2" gate="G$1" pin="GND_B"/>
 <wire x1="251.46" y1="127" x2="251.46" y2="124.46" width="0.1524" layer="91"/>
 <wire x1="251.46" y1="124.46" x2="251.46" y2="116.84" width="0.1524" layer="91"/>
 <wire x1="243.84" y1="127" x2="251.46" y2="127" width="0.1524" layer="91"/>
 <junction x="251.46" y="127"/>
-<pinref part="X1" gate="G$1" pin="GND_H"/>
+<pinref part="J2" gate="G$1" pin="GND_H"/>
 <wire x1="243.84" y1="124.46" x2="251.46" y2="124.46" width="0.1524" layer="91"/>
 <junction x="251.46" y="124.46"/>
@@
 <wire x1="76.2" y1="48.26" x2="27.94" y2="48.26" width="0.1524" layer="91"/>
 <wire x1="27.94" y1="48.26" x2="27.94" y2="58.42" width="0.1524" layer="91"/>
-<pinref part="X2" gate="G$1" pin="GND"/>
+<pinref part="X1" gate="G$1" pin="GND"/>
 <wire x1="27.94" y1="58.42" x2="30.48" y2="58.42" width="0.1524" layer="91"/>
 <pinref part="GND8" gate="1" pin="GND"/>
@@
 <wire x1="76.2" y1="12.7" x2="27.94" y2="12.7" width="0.1524" layer="91"/>
 <wire x1="27.94" y1="12.7" x2="27.94" y2="22.86" width="0.1524" layer="91"/>
-<pinref part="X3" gate="G$1" pin="GND"/>
+<pinref part="X2" gate="G$1" pin="GND"/>
 <wire x1="27.94" y1="22.86" x2="30.48" y2="22.86" width="0.1524" layer="91"/>
 <pinref part="GND9" gate="1" pin="GND"/>
@@
 <net name="+3V3" class="0">
 <segment>
-<pinref part="X1" gate="G$1" pin="3V3_A"/>
+<pinref part="J2" gate="G$1" pin="3V3_A"/>
 <pinref part="+3V1" gate="G$1" pin="+3V3"/>
 <wire x1="233.68" y1="152.4" x2="233.68" y2="157.48" width="0.1524" layer="91"/>
@@
 </segment>
 <segment>
-<pinref part="X2" gate="G$1" pin="VDD"/>
+<pinref part="X1" gate="G$1" pin="VDD"/>
 <wire x1="60.96" y1="60.96" x2="76.2" y2="60.96" width="0.1524" layer="91"/>
 <pinref part="+3V3" gate="G$1" pin="+3V3"/>
@@
 </segment>
 <segment>
-<pinref part="X3" gate="G$1" pin="VDD"/>
+<pinref part="X2" gate="G$1" pin="VDD"/>
 <wire x1="60.96" y1="25.4" x2="76.2" y2="25.4" width="0.1524" layer="91"/>
 <pinref part="+3V4" gate="G$1" pin="+3V3"/>
@@
 <net name="BCLK" class="0">
 <segment>
-<pinref part="X1" gate="G$1" pin="GPIO18"/>
+<pinref part="J2" gate="G$1" pin="GPIO18"/>
 <wire x1="213.36" y1="137.16" x2="203.2" y2="137.16" width="0.1524" layer="91"/>
 <label x="203.2" y="137.16" size="1.778" layer="95"/>
@@
 <net name="LRCLK" class="0">
 <segment>
-<pinref part="X1" gate="G$1" pin="GPIO19"/>
+<pinref part="J2" gate="G$1" pin="GPIO19"/>
 <wire x1="213.36" y1="129.54" x2="203.2" y2="129.54" width="0.1524" layer="91"/>
 <label x="203.2" y="129.54" size="1.778" layer="95"/>
@@
 <net name="DATA" class="0">
 <segment>
-<pinref part="X1" gate="G$1" pin="GPIO21"/>
+<pinref part="J2" gate="G$1" pin="GPIO21"/>
 <wire x1="213.36" y1="119.38" x2="203.2" y2="119.38" width="0.1524" layer="91"/>
 <label x="203.2" y="119.38" size="1.778" layer="95"/>
@@
 <net name="SCL" class="0">
 <segment>
-<pinref part="X1" gate="G$1" pin="SCL"/>
+<pinref part="J2" gate="G$1" pin="SCL"/>
 <wire x1="213.36" y1="114.3" x2="203.2" y2="114.3" width="0.1524" layer="91"/>
 <label x="203.2" y="114.3" size="1.778" layer="95"/>
@@
 <net name="SDA" class="0">
 <segment>
-<pinref part="X1" gate="G$1" pin="SDA"/>
+<pinref part="J2" gate="G$1" pin="SDA"/>
 <wire x1="213.36" y1="111.76" x2="203.2" y2="111.76" width="0.1524" layer="91"/>
 <label x="203.2" y="111.76" size="1.778" layer="95"/>
@@
 </segment>
 <segment>
-<pinref part="X2" gate="G$1" pin="OUT"/>
+<pinref part="X1" gate="G$1" pin="OUT"/>
 <wire x1="60.96" y1="58.42" x2="71.12" y2="58.42" width="0.1524" layer="91"/>
 <label x="71.12" y="58.42" size="1.778" layer="95" rot="MR0"/>
 </segment>
 <segment>
-<pinref part="X3" gate="G$1" pin="OUT"/>
+<pinref part="X2" gate="G$1" pin="OUT"/>
 <wire x1="60.96" y1="22.86" x2="71.12" y2="22.86" width="0.1524" layer="91"/>
 <label x="71.12" y="22.86" size="1.778" layer="95" rot="MR0"/>
@@
 </segment>
 <segment>
-<pinref part="X2" gate="G$1" pin="EN"/>
+<pinref part="X1" gate="G$1" pin="EN"/>
 <wire x1="30.48" y1="60.96" x2="20.32" y2="60.96" width="0.1524" layer="91"/>
 <label x="20.32" y="60.96" size="1.778" layer="95"/>
@@
 </segment>
 <segment>
-<pinref part="X3" gate="G$1" pin="EN"/>
+<pinref part="X2" gate="G$1" pin="EN"/>
 <wire x1="30.48" y1="25.4" x2="20.32" y2="25.4" width="0.1524" layer="91"/>
 <label x="20.32" y="25.4" size="1.778" layer="95"/>

Commit message: fix minor probrems, and add scripts to generate decal image for 3D rendering
Connections:
- net EN41 renamed EN44
Changed lines of the file:
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@@
-</segment>
-</net>
-<net name="EN41" class="0">
-<segment>
-<pinref part="U1" gate="G$1" pin="GPIO6"/>
-<wire x1="109.22" y1="109.22" x2="121.92" y2="109.22" width="0.1524" layer="91"/>
-<label x="121.92" y="109.22" size="1.778" layer="95" rot="MR0"/>
-</segment>
-<segment>
-<pinref part="X1" gate="G$1" pin="EN"/>
-<wire x1="30.48" y1="60.96" x2="20.32" y2="60.96" width="0.1524" layer="91"/>
-<label x="20.32" y="60.96" size="1.778" layer="95"/>
 </segment>
 </net>
@@
 </segment>
 </net>
+<net name="EN44" class="0">
+<segment>
+<pinref part="X1" gate="G$1" pin="EN"/>
+<wire x1="30.48" y1="60.96" x2="20.32" y2="60.96" width="0.1524" layer="91"/>
+<label x="20.32" y="60.96" size="1.778" layer="95"/>
+</segment>
+<segment>
+<pinref part="U1" gate="G$1" pin="GPIO6"/>
+<wire x1="109.22" y1="109.22" x2="121.92" y2="109.22" width="0.1524" layer="91"/>
+<label x="121.92" y="109.22" size="1.778" layer="95" rot="MR0"/>
+</segment>
+</net>
