File: pcb/type2/sonopi-dac-type2.sch (EAGLE design)
At the start: 25 parts, among them J1 HLR-3201VXB-004HG, J2 HLR-3201VXB-003HG, J3 RASPI_BOARD_B+#_ZERO, U1 PCM5122PW, U2 MCP1703AT-3302E/CB, X1 22.5792MHz, X2 24.576MHz

Commit message: change footprint of 3225 oscillator
Parts:
- X1, X2: device oscillator:OSC-3225 -> oscillator:OSC-3225HS
Changed lines of the file:
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@@
 <?xml version="1.0" encoding="utf-8"?>
 <!DOCTYPE eagle SYSTEM "eagle.dtd">
-<eagle version="9.5.2">
+<eagle version="9.6.1">
 <drawing>
 <settings>
@@
 <part name="C10" library="rcl" library_urn="urn:adsk.eagle:library:334" deviceset="C-EU" device="C0805" package3d_urn="urn:adsk.eagle:package:23617/2" value="2.2uF/25V"/>
 <part name="R1" library="rcl" library_urn="urn:adsk.eagle:library:334" deviceset="R-US_" device="R0603" package3d_urn="urn:adsk.eagle:package:23555/3" value="470Ω"/>
-<part name="X1" library="oscillator" library_urn="urn:adsk.eagle:library:15275959" deviceset="OSC" device="-3225" package3d_urn="urn:adsk.eagle:package:15275963/2" value="22.5792MHz"/>
+<part name="X1" library="oscillator" library_urn="urn:adsk.eagle:library:15275959" deviceset="OSC" device="-3225HS" package3d_urn="urn:adsk.eagle:package:20544451/2" value="22.5792MHz"/>
 <part name="+3V3" library="supply1" library_urn="urn:adsk.eagle:library:371" deviceset="+3V3" device=""/>
 <part name="C13" library="rcl" library_urn="urn:adsk.eagle:library:334" deviceset="C-EU" device="C0603" package3d_urn="urn:adsk.eagle:package:23616/2" value="0.1uF/100V"/>
 <part name="GND8" library="supply1" library_urn="urn:adsk.eagle:library:371" deviceset="GND" device=""/>
-<part name="X2" library="oscillator" library_urn="urn:adsk.eagle:library:15275959" deviceset="OSC" device="-3225" package3d_urn="urn:adsk.eagle:package:15275963/2" value="24.576MHz"/>
+<part name="X2" library="oscillator" library_urn="urn:adsk.eagle:library:15275959" deviceset="OSC" device="-3225HS" package3d_urn="urn:adsk.eagle:package:20544451/2" value="24.576MHz"/>
 <part name="+3V4" library="supply1" library_urn="urn:adsk.eagle:library:371" deviceset="+3V3" device=""/>
 <part name="C14" library="rcl" library_urn="urn:adsk.eagle:library:334" deviceset="C-EU" device="C0603" package3d_urn="urn:adsk.eagle:package:23616/2" value="0.1uF/100V"/>
